File: Flight Tracker PCB/Flight Tracker/_saved_Flight Tracker.sch (KiCad schematic (older format))
At the start: 17 parts, among them J1 Conn_01x02, Q1 BSS138, Q2 BSS138, U1 NTX2, U2 UBlox_MAX8

Commit message: Made a few symbols and footprints for the BH1750, Ublox8, and BMP280
Parts:
- added U?: BMP280, NTX2:BMP280, symbol NTX2:BMP280
- added U?: BH1750, NTX2:BH1750, symbol NTX2:BH1750
- U2: footprint (none) -> NTX2:Ublox Max 8
Changed lines of the file:
@@
 F 0 "U2" H 7191 5496 50  0000 L CNN
 F 1 "UBlox_MAX8" H 7191 5405 50  0000 L CNN
-F 2 "" H 6900 6600 50  0001 C CNN
+F 2 "NTX2:Ublox Max 8" H 6900 6600 50  0001 C CNN
 F 3 "" H 6900 6600 50  0001 C CNN
 	1    6500 5450
@@
 Wire Wire Line
 	6750 2350 6750 2300
+$Comp
+L NTX2:BMP280 U?
+U 1 1 5E93A3D7
+P 4200 5400
+F 0 "U?" H 4200 5903 50  0000 C CNN
+F 1 "BMP280" H 4200 5812 50  0000 C CNN
+F 2 "NTX2:BMP280" H 3800 5875 50  0001 C CNN
+F 3 "" H 3800 5875 50  0001 C CNN
+	1    4200 5400
+	1    0    0    -1
+$EndComp
+$Comp
+L NTX2:BH1750 U?
+U 1 1 5E93BA38
+P 3200 5850
+F 0 "U?" H 3200 6315 50  0000 C CNN
+F 1 "BH1750" H 3200 6224 50  0000 C CNN
+F 2 "NTX2:BH1750" H 2500 6300 50  0001 C CNN
+F 3 "" H 2500 6300 50  0001 C CNN
+	1    3200 5850
+	1    0    0    -1
+$EndComp
 $EndSCHEMATC
