File: Flight Tracker PCB/Flight Tracker/_saved_Flight Tracker.sch (KiCad schematic (older format))
At the start: 53 parts, among them J1 Screw_Terminal_01x02, J2 Conn_01x02, J3 Conn_01x02, J4 Conn_02x03_Odd_Even, J5 Conn_01x02, Q1 FQP47P06, Q2 BSS138, Q3 BSS138, Q4 BSS138, Q5 BSS138, Q6 BSS138, Q7 BSS138, Q8 BSS138, Q9 BSS138, U1 NTX2, U2 UBlox_MAX8, U3 BH1750, U4 MPU_9250, U5 ML8511, U6 BMP280, U7 SMA_5pin, U8 UM232R

Commit message: created draft pcb, decided that removing the um232r footprint is required to make the pcb look nicer
Parts:
- A1: footprint Module:Arduino_UNO_R3 -> NTX2:Arduino_UNO_R3_(Headers_Version)
Changed lines of the file:
@@
 F 0 "A1" H 10500 5575 50  0000 C CNN
 F 1 "Arduino_UNO_R3" H 11350 3525 50  0000 C CNN
-F 2 "Module:Arduino_UNO_R3" H 11000 3575 50  0001 L CNN
+F 2 "NTX2:Arduino_UNO_R3_(Headers_Version)" H 11000 3575 50  0001 L CNN
 F 3 "https://www.arduino.cc/en/Main/arduinoBoardUno" H 10650 5675 50  0001 C CNN
 	1    10850 4625
