File: Flight Tracker PCB/Flight Tracker/Flight Tracker.sch (KiCad schematic (older format))
At the start: 17 parts, among them J1 Conn_01x02, Q1 BSS138, Q2 BSS138, U1 NTX2, U2 UBlox_MAX8

Commit message: Created ML8511, MPU9250_MS5611 symbols and footprints
Parts:
- added U?: BMP280, NTX2:BMP280, symbol NTX2:BMP280
- added U?: BH1750, NTX2:BH1750, symbol NTX2:BH1750
- added U?: ML8511, NTX2:ML8511, symbol NTX2:ML8511
- added U?: MPU-9250_MS5611, NTX2:MPU9250_MS5611, symbol NTX2:MPU-9250_MS5611
- U2: footprint (none) -> NTX2:Ublox Max 8
Changed lines of the file:
@@
 F 0 "U2" H 7191 5496 50  0000 L CNN
 F 1 "UBlox_MAX8" H 7191 5405 50  0000 L CNN
-F 2 "" H 6900 6600 50  0001 C CNN
+F 2 "NTX2:Ublox Max 8" H 6900 6600 50  0001 C CNN
 F 3 "" H 6900 6600 50  0001 C CNN
 	1    6500 5450
@@
 Wire Wire Line
 	6750 2350 6750 2300
+$Comp
+L NTX2:BMP280 U?
+U 1 1 5E93A3D7
+P 4200 5400
+F 0 "U?" H 4200 5903 50  0000 C CNN
+F 1 "BMP280" H 4200 5812 50  0000 C CNN
+F 2 "NTX2:BMP280" H 3800 5875 50  0001 C CNN
+F 3 "" H 3800 5875 50  0001 C CNN
+	1    4200 5400
+	1    0    0    -1
+$EndComp
+$Comp
+L NTX2:BH1750 U?
+U 1 1 5E93BA38
+P 3200 5850
+F 0 "U?" H 3200 6315 50  0000 C CNN
+F 1 "BH1750" H 3200 6224 50  0000 C CNN
+F 2 "NTX2:BH1750" H 2500 6300 50  0001 C CNN
+F 3 "" H 2500 6300 50  0001 C CNN
+	1    3200 5850
+	1    0    0    -1
+$EndComp
+$Comp
+L NTX2:ML8511 U?
+U 1 1 5E93CEA8
+P 4875 6200
+F 0 "U?" H 4875 6615 50  0000 C CNN
+F 1 "ML8511" H 4875 6524 50  0000 C CNN
+F 2 "NTX2:ML8511" H 4125 6500 50  0001 C CNN
+F 3 "" H 4125 6500 50  0001 C CNN
+	1    4875 6200
+	1    0    0    -1
+$EndComp
+$Comp
+L NTX2:MPU-9250_MS5611 U?
+U 1 1 5E93E221
+P 4025 6450
+F 0 "U?" H 4025 6915 50  0000 C CNN
+F 1 "MPU-9250_MS5611" H 4025 6824 50  0000 C CNN
+F 2 "NTX2:MPU9250_MS5611" H 3700 6800 50  0001 C CNN
+F 3 "" H 3700 6800 50  0001 C CNN
+	1    4025 6450
+	1    0    0    -1
+$EndComp
 $EndSCHEMATC

Commit message: Attempted to wire the BMP280 correctly cross referencing the datasheet
Parts:
- added Q3, Q4: BSS138, Package_TO_SOT_SMD:SOT-23, symbol Transistor_FET:BSS138
- added R10, R11, R12, R13: 10K, symbol Device:R
- gave numbers to parts that had none: 4
Connections:
- net labels added: BMP280_SCL_3V3, BMP280_SDA_3V3, Ublox_SCL_3V3, Ublox_SDA_3V3, Ublox­_SCL_3V3
- net labels removed: SCL_3V3, SDA_3V3
- wire segments 55 -> 79
Other:
- note added: "BMP280 SCL Shifter"
- note added: "BMP280 SDA Shifter"
- note added: "CSB -> Chip Select Pull up for I2C, pull down for SPI\nSDO -> Conn to GND gives 0x76 adress \nand conn (don't leave floating) to VCC gives 0x77 address"
- note added: "I2C Bus"
- note added: "Ublox SCL Shifter"
- note added: "Ublox SDA Shifter"
- note removed: "I2C Line Level Shifters"
- note removed: "Ublox Bus"
