File: Flight Tracker PCB/Flight Tracker/Flight Tracker.sch (KiCad schematic (older format))
At the start: 41 parts, among them J1 Conn_01x02, Q1 BSS138, Q2 BSS138, Q3 BSS138, Q4 BSS138, Q5 BSS138, Q6 BSS138, Q7 BSS138, Q8 BSS138, U1 NTX2, U2 UBlox_MAX8, U3 BH1750, U4 MPU_9250, U5 ML8511, U6 BMP280

Commit message: Implemented reverse voltage protection at VIN using FQP47P06 (p-channel mosfet with high gate-drain voltage
Parts:
- removed Q1, Q2: BSS138, Package_TO_SOT_SMD:SOT-23, symbol Transistor_FET:BSS138
- removed R1, R2, R3, R4: 10K, symbol Device:R
- added BZ1: Buzzer, symbol Device:Buzzer
- added J2: Conn_01x02, symbol Connector_Generic:Conn_01x02
- added Q1: FQP47P06, TO254P483X1016X2261-3P, symbol FQP47P06:FQP47P06
- added RV1: R_POT, symbol Device:R_POT
- added U7: SMA_5pin, NTX2:SMA_EDGE, symbol NTX2:SMA_5pin
- D1, D2: footprint (none) -> LED_SMD:LED_1206_3216Metric_Pad1.42x1.75mm_HandSolder
- J1: footprint (none) -> Connector_PinSocket_2.54mm:PinSocket_1x02_P2.54mm_Vertical
- R10, R11, R12, R13, R14, R15, R16, R17, R18, R19, R20, R21, R22, R23, R5, R6, R8, R9: footprint (none) -> Resistor_SMD:R_1206_3216Metric_Pad1.42x1.75mm_HandSolder
- R7: value 47K -> 10K; footprint (none) -> Resistor_SMD:R_1206_3216Metric_Pad1.42x1.75mm_HandSolder
Connections:
- net labels removed: RADIO_PIN, Ublox_SDA_3V3, Ublox­_SCL_3V3
- wire segments 141 -> 148
- no-connect marks 31 -> 27
Other:
- note added: "50 Ohm SMA edge\nmounted antenna \nconnector for \n164mm 1/4 wave \npigtail"
- note added: "Reverse voltage protection\nusing p-channel mosfet\n"
- note added: "SCL -> I2C Clock (Unused, only for I2C interface)\nSDA -> I2C Data (Unused, only for I2C interface)\nTP -> Time Pulse Output (NC)\nVCC -> 3V3 Supply\nGND -> GND\nNC -> NC\nTXD -> Con to MC RX\nRXD - > Con to MC TX\n"
- note added: "The fixed 10K ensures atleast 10K of resistance minimum.\nThe pot will allow tuning of the frequency shift"
- note added: "UART Connections\n"
- note added: "When configured as a pass through you\nneed a voltage divider between arduino RX\nand ublox RX to convert the 5v arduino logic\nto 3.3V. Set R1=1K and R2=2"
- note removed: "SCL -> I2C Clock\nSDA -> I2C Data\nTP -> Time Pulse Output (NC)\nVCC -> 3V3 Supply\nGND -> GND\nNC -> NC\nTXD -> Con to MC RX\nRXD - > Con to MC TX\n"
- note removed: "Ublox SCL Shifter"
- note removed: "Ublox SDA Shifter"

Commit message: created footprint for buzzer and corrected it's symbol incorrect wiring
Parts:
- added F1: 500mA Fuse, symbol Device:Fuse_Small
- BZ1: footprint (none) -> NTX2:5V_Buzzer
- Q1: footprint TO254P483X1016X2261-3P -> NTX2:TO254P483X1016X2261-3P
Connections:
- wire segments 148 -> 150
Other:
- note added: "Precautionary fuse to prevent excess \ncurrent draw from damaging circuit\n"
Changed lines of the file:
@@
 L Connector_Generic:Conn_01x02 J1
 U 1 1 5E90A2FC
-P 10750 2200
-F 0 "J1" V 10716 2012 50  0000 R CNN
-F 1 "Conn_01x02" V 10800 2025 50  0000 R CNN
-F 2 "Connector_PinSocket_2.54mm:PinSocket_1x02_P2.54mm_Vertical" H 10750 2200 50  0001 C CNN
-F 3 "~" H 10750 2200 50  0001 C CNN
-	1    10750 2200
+P 10750 1925
+F 0 "J1" V 10716 1737 50  0000 R CNN
+F 1 "Conn_01x02" V 10800 1750 50  0000 R CNN
+F 2 "Connector_PinSocket_2.54mm:PinSocket_1x02_P2.54mm_Vertical" H 10750 1925 50  0001 C CNN
+F 3 "~" H 10750 1925 50  0001 C CNN
+	1    10750 1925
 	0    -1   -1   0
 $EndComp
-Text Notes 10400 2075 0    50   ~ 0
+Text Notes 10425 1800 0    50   ~ 0
 Power Supply (6-24V)\n
 NoConn ~ 11700 6900
@@
 Wire Wire Line
 	10700 3425 10750 3425
-Connection ~ 10750 3425
 Wire Wire Line
 	10750 3425 10750 3625
@@
 Wire Wire Line
 	7000 9375 7000 9400
-Text Notes 6425 10825 0    50   ~ 0
+Text Notes 6300 10875 0    50   ~ 0
 Resistive voltage sensor using potenial divider\nconnected to battery source. \nInput (V_S_I) conn to VIN terminals\nOutput (V_S_O) conn to A0 of MC
 NoConn ~ 10350 4625
@@
 F 0 "BZ1" H 10000 4625 50  0000 C CNN
 F 1 "Buzzer" H 10375 4625 50  0000 C CNN
-F 2 "" V 10075 4725 50  0001 C CNN
+F 2 "NTX2:5V_Buzzer" V 10075 4725 50  0001 C CNN
 F 3 "~" V 10075 4725 50  0001 C CNN
 	1    10100 4625
-	-1   0    0    1
+	-1   0    0    -1
 $EndComp
 $Comp
@@
 F 0 "Q1" H 10879 2771 50  0000 L CNN
 F 1 "FQP47P06" H 10879 2680 50  0000 L CNN
-F 2 "TO254P483X1016X2261-3P" H 10900 2575 50  0001 L CNN
+F 2 "NTX2:TO254P483X1016X2261-3P" H 10900 2575 50  0001 L CNN
 F 3 "https://www.onsemi.com/pub/Collateral/FQP47P06-D.pdf" H 10900 2475 50  0001 L CNN
 F 4 "Trans MOSFET P-CH 60V 47A 3-Pin TO-220" H 10900 2375 50  0001 L CNN "Description"
@@
 Wire Wire Line
 	10375 2625 10450 2625
-Wire Wire Line
-	10750 3025 10750 3200
 $Comp
 L power:PWR_FLAG #FLG0103
@@
 	0    1    1    0
 $EndComp
-Connection ~ 10750 3200
-Wire Wire Line
-	10750 3200 10750 3425
-Wire Wire Line
-	10750 2400 10750 2425
-Wire Wire Line
-	10850 2400 10850 2425
+Wire Wire Line
+	10750 2125 10750 2150
+Wire Wire Line
+	10850 2125 10850 2400
 Wire Wire Line
 	9850 5950 9850 5975
-Wire Bus Line
-	5850 4550 5850 10675
-Wire Bus Line
-	5900 4550 5900 10675
 $Comp
 L power:PWR_FLAG #FLG0104
@@
 $EndComp
 Connection ~ 10850 2400
+$Comp
+L Device:Fuse_Small F1
+U 1 1 5E9D748E
+P 10750 2250
+F 0 "F1" V 10675 2125 50  0000 L CNN
+F 1 "500mA Fuse" V 10750 2375 50  0000 L CNN
+F 2 "" H 10750 2250 50  0001 C CNN
+F 3 "~" H 10750 2250 50  0001 C CNN
+	1    10750 2250
+	0    1    1    0
+$EndComp
+Wire Wire Line
+	10850 2400 10850 2425
+Wire Wire Line
+	10750 2350 10750 2425
+Text Notes 9200 2350 0    50   ~ 0
+Precautionary fuse to prevent excess \ncurrent draw from damaging circuit\n
+Wire Bus Line
+	5850 4550 5850 10675
+Wire Bus Line
+	5900 4550 5900 10675
+Connection ~ 10750 3425
+Wire Wire Line
+	10750 3200 10750 3425
+Connection ~ 10750 3200
+Wire Wire Line
+	10750 3025 10750 3200
 $EndSCHEMATC

Commit message: First bit of good progress on transmitting the NMEA messages parsed using tinyGPS++, also added PUBX commands to turn off unwanted NMEA messages as we only care for GNGGA messages for HAB
Parts:
- added D3: GPS_LOCK, LED_SMD:LED_1206_3216Metric_Pad1.42x1.75mm_HandSolder, symbol Device:LED
- added R1: 150R, Resistor_SMD:R_1206_3216Metric_Pad1.42x1.75mm_HandSolder, symbol Device:R
- F1: footprint (none) -> NTX2:MC000827
Connections:
- wire segments 150 -> 154
- no-connect marks 27 -> 26
Changed lines of the file:
@@
 Text Label 7225 6725 0    50   ~ 0
 UV_OUT
-Text Label 10350 4425 2    50   ~ 0
+Text Label 10350 4525 2    50   ~ 0
 UV_OUT
 $Comp
@@
 Text Notes 6300 10875 0    50   ~ 0
 Resistive voltage sensor using potenial divider\nconnected to battery source. \nInput (V_S_I) conn to VIN terminals\nOutput (V_S_O) conn to A0 of MC
-NoConn ~ 10350 4625
 NoConn ~ 10350 4725
 NoConn ~ 10350 4825
@@
 L Device:Buzzer BZ1
 U 1 1 5EED2E18
-P 10100 4625
-F 0 "BZ1" H 10000 4625 50  0000 C CNN
-F 1 "Buzzer" H 10375 4625 50  0000 C CNN
-F 2 "NTX2:5V_Buzzer" V 10075 4725 50  0001 C CNN
-F 3 "~" V 10075 4725 50  0001 C CNN
-	1    10100 4625
+P 10100 4725
+F 0 "BZ1" H 10000 4725 50  0000 C CNN
+F 1 "Buzzer" H 10125 4575 50  0000 C CNN
+F 2 "NTX2:5V_Buzzer" V 10075 4825 50  0001 C CNN
+F 3 "~" V 10075 4825 50  0001 C CNN
+	1    10100 4725
 	-1   0    0    -1
 $EndComp
@@
 L power:GND #PWR015
 U 1 1 5EEF331B
-P 10250 4775
-F 0 "#PWR015" H 10250 4525 50  0001 C CNN
-F 1 "GND" H 10255 4602 50  0000 C CNN
-F 2 "" H 10250 4775 50  0001 C CNN
-F 3 "" H 10250 4775 50  0001 C CNN
-	1    10250 4775
-	1    0    0    -1
-$EndComp
-Wire Wire Line
-	10250 4775 10250 4725
-Wire Wire Line
-	10250 4725 10200 4725
+P 10250 4875
+F 0 "#PWR015" H 10250 4625 50  0001 C CNN
+F 1 "GND" H 10255 4702 50  0000 C CNN
+F 2 "" H 10250 4875 50  0001 C CNN
+F 3 "" H 10250 4875 50  0001 C CNN
+	1    10250 4875
+	1    0    0    -1
+$EndComp
+Wire Wire Line
+	10250 4875 10250 4825
+Wire Wire Line
+	10250 4825 10200 4825
 Text GLabel 9575 5550 2    50   Input ~ 0
 5V
@@
 $EndComp
 Wire Wire Line
-	10200 4525 10350 4525
+	10200 4625 10350 4625
 Wire Wire Line
 	9600 4325 9600 4100
@@
 F 0 "F1" V 10675 2125 50  0000 L CNN
 F 1 "500mA Fuse" V 10750 2375 50  0000 L CNN
-F 2 "" H 10750 2250 50  0001 C CNN
+F 2 "NTX2:MC000827" H 10750 2250 50  0001 C CNN
 F 3 "~" H 10750 2250 50  0001 C CNN
 	1    10750 2250
@@
 Text Notes 9200 2350 0    50   ~ 0
 Precautionary fuse to prevent excess \ncurrent draw from damaging circuit\n
+Connection ~ 10750 3425
+Wire Wire Line
+	10750 3200 10750 3425
+Connection ~ 10750 3200
+Wire Wire Line
+	10750 3025 10750 3200
+$Comp
+L Device:R R1
+U 1 1 5E9FC6AB
+P 9900 4425
+F 0 "R1" V 9850 4575 50  0000 L CNN
+F 1 "150R" V 10000 4325 50  0000 L CNN
+F 2 "Resistor_SMD:R_1206_3216Metric_Pad1.42x1.75mm_HandSolder" V 9830 4425 50  0001 C CNN
+F 3 "~" H 9900 4425 50  0001 C CNN
+	1    9900 4425
+	0    1    1    0
+$EndComp
+Wire Wire Line
+	10050 4425 10350 4425
+$Comp
+L Device:LED D3
+U 1 1 5EA024F7
+P 9600 4600
+F 0 "D3" V 9500 4600 50  0000 L CNN
+F 1 "GPS_LOCK" V 9600 4175 50  0000 L CNN
+F 2 "LED_SMD:LED_1206_3216Metric_Pad1.42x1.75mm_HandSolder" H 9600 4600 50  0001 C CNN
+F 3 "~" H 9600 4600 50  0001 C CNN
+	1    9600 4600
+	0    -1   -1   0
+$EndComp
+$Comp
+L power:GND #PWR018
+U 1 1 5EA0E79C
+P 9600 4800
+F 0 "#PWR018" H 9600 4550 50  0001 C CNN
+F 1 "GND" H 9605 4627 50  0000 C CNN
+F 2 "" H 9600 4800 50  0001 C CNN
+F 3 "" H 9600 4800 50  0001 C CNN
+	1    9600 4800
+	1    0    0    -1
+$EndComp
+Wire Wire Line
+	9600 4800 9600 4750
+Wire Wire Line
+	9600 4450 9600 4425
+Wire Wire Line
+	9600 4425 9750 4425
+Wire Bus Line
+	5900 4550 5900 10675
 Wire Bus Line
 	5850 4550 5850 10675
-Wire Bus Line
-	5900 4550 5900 10675
-Connection ~ 10750 3425
-Wire Wire Line
-	10750 3200 10750 3425
-Connection ~ 10750 3200
-Wire Wire Line
-	10750 3025 10750 3200
 $EndSCHEMATC

Commit message: implemented UV sensor, took out carrier shift pot (47k res instead), changed UV_OUT pin, some other stuff, added level shifter for ublox gps tcd and rxd lines, added low voltage detection,\n added no gps data reset function to attempt to fix problem
Parts:
- removed RV1: R_POT, symbol Device:R_POT
- added Q2, Q9: BSS138, Package_TO_SOT_SMD:SOT-23, symbol Transistor_FET:BSS138
- added R2, R24, R3, R4: 10K, Resistor_SMD:R_1206_3216Metric_Pad1.42x1.75mm_HandSolder, symbol Device:R
- R7: value 10K -> 47k
Connections:
- net labels added: Ublox_RXD_3V3, Ublox_RXD_5V, Ublox_TXD_3V3, Ublox_TXD_5V
- wire segments 154 -> 181
- no-connect marks 26 -> 21
Other:
- note added: "!UV 3V3 Reference!"

Commit message: added ICSP header on PCB, added connector for external thermistor with voltage divider to A3, added connector to tap into I2c bus
Parts:
- removed J1: Conn_01x02, Connector_PinSocket_2.54mm:PinSocket_1x02_P2.54mm_Vertical, symbol Connector_Generic:Conn_01x02
- added J1: Screw_Terminal_01x02, NTX2:2_Pin_Screw_Terminal, symbol Connector:Screw_Terminal_01x02
- added J3: Conn_01x02, Connector_JST:JST_EH_B02B-EH-A_1x02_P2.50mm_Vertical, symbol Connector_Generic:Conn_01x02
- added J4: Conn_02x03_Odd_Even, Connector_PinHeader_2.54mm:PinHeader_2x03_P2.54mm_Vertical, symbol Connector_Generic:Conn_02x03_Odd_Even
- added J5: Conn_01x02, symbol Connector_Generic:Conn_01x02
- added R25: 100k, Resistor_SMD:R_1206_3216Metric_Pad1.42x1.75mm_HandSolder, symbol Device:R
- added U8: UM232R, NTX2:UM232R_1, symbol UM232R:UM232R
- J2: footprint (none) -> Connector_PinSocket_2.54mm:PinSocket_1x02_P2.54mm_Vertical
Connections:
- net labels added: +5V, MISO, MOSI, RST, SCK, Thermistor, UM232R_RXD, UM232R_TXD
- wire segments 181 -> 203
- no-connect marks 21 -> 18
Other:
- note added: "External UART module needed\nfor debugging software serial\n(harware serial occupied by GPS)"
- note added: "ICSP Header for programming arduino\n(original blocked by tracker sheild)"
- note added: "Tap into \nI2C lines\n(no pullups)"
- note added: "Thermistor connector for\nexternal temperature sensor\n(with voltage 1:1 divider)"

Commit message: created draft pcb, decided that removing the um232r footprint is required to make the pcb look nicer
Parts:
- J5: footprint (none) -> Connector_JST:JST_EH_B02B-EH-A_1x02_P2.50mm_Vertical
Connections:
- wire segments 203 -> 207
Changed lines of the file:
@@
 	5750 7075 5850 7175
 Wire Wire Line
-	5750 7075 4750 7075
+	5750 7075 5725 7075
 Connection ~ 4750 7075
 Entry Wire Line
@@
 Connection ~ 5600 6000
 Wire Wire Line
-	5600 6000 5800 6000
-Wire Wire Line
 	5575 4625 5575 4825
 Connection ~ 5575 4825
@@
 F 0 "J5" H 5425 6500 50  0000 C CNN
 F 1 "Conn_01x02" H 5425 6825 50  0000 C CNN
-F 2 "" H 5425 6700 50  0001 C CNN
+F 2 "Connector_JST:JST_EH_B02B-EH-A_1x02_P2.50mm_Vertical" H 5425 6700 50  0001 C CNN
 F 3 "~" H 5425 6700 50  0001 C CNN
 	1    5425 6700
 	-1   0    0    1
 $EndComp
-Entry Wire Line
-	5750 6700 5850 6800
-Entry Wire Line
-	5800 6600 5900 6700
-Wire Wire Line
-	5800 6600 5625 6600
-Wire Wire Line
-	5750 6700 5625 6700
+Text Notes 5950 6775 0    50   ~ 0
+Tap into \nI2C lines\n(no pullups)
+Wire Wire Line
+	5625 6600 5725 6600
+Wire Wire Line
+	5625 6700 5725 6700
+Wire Wire Line
+	5725 6700 5725 7075
+Connection ~ 5725 7075
+Wire Wire Line
+	5725 7075 4750 7075
+Wire Wire Line
+	5725 6600 5725 6000
+Wire Wire Line
+	5600 6000 5725 6000
+Connection ~ 5725 6000
+Wire Wire Line
+	5725 6000 5800 6000
 Wire Bus Line
 	5900 4550 5900 10675
 Wire Bus Line
 	5850 4550 5850 10675
-Text Notes 5950 6775 0    50   ~ 0
-Tap into \nI2C lines\n(no pullups)
 $EndSCHEMATC
